Commit message: changed plugin to control force and small fixes to model

File: environment/rrbot_description/urdf/rrbot.xacro (robot description, xacro)
@@ -4,10 +4,8 @@
   <!-- Constants for robot dimensions -->
   <xacro:property name="PI" value="3.1415926535897931"/>
-  <xacro:property name="mass" value="1" /> <!-- arbitrary value for mass -->
+  <xacro:property name="mass" value="0.2" /> <!-- arbitrary value for mass -->
   <xacro:property name="width" value="0.1" /> <!-- Square dimensions (widthxwidth) of beams -->
-  <xacro:property name="height1" value="2" /> <!-- Link 1 -->
-  <xacro:property name="height2" value="1" /> <!-- Link 2 -->
-  <xacro:property name="height3" value="1" /> <!-- Link 3 -->
-  <xacro:property name="camera_link" value="0.05" /> <!-- Size of square 'camera' box -->
+  <xacro:property name="height1" value="1.1" /> <!-- Link 1 -->
+  <xacro:property name="height2" value="0.6" /> <!-- Link 2 -->
   <xacro:property name="axel_offset" value="0.05" /> <!-- Space btw top of beam and the each joint -->
   <!-- Import all Gazebo-customization elements, including Gazebo colors -->
@@ -32,5 +30,5 @@
     <inertial>
       <origin xyz="0 0 0.02" rpy="0 0 0"/>
-      <mass value="1000"/>
+      <mass value="0.5"/>
       <inertia ixx="1000" ixy="1000" ixz="1000" iyy="1000" iyz="1000" izz="1000" />
     </inertial>
@@ -43,23 +41,4 @@
     <limit velocity="10000" effort="10000" lower="-10" upper="10" />
   </joint>
- <!-- link name="base_1">
-   <visual>
-      <origin xyz="1 0 1.51" rpy="0 0 0" />
-      <geometry>
-        <box size="0.1 2.1 3" />
-      </geometry>
-    </visual>
-   <collision>
-      <origin xyz="1 0 1.51" rpy="0 0 0" />
-      <geometry>
-        <box size="0.1 2.1 3" />
-      </geometry>
-    </collision>
-  </link >
-  <joint name="f_1" type="fixed">
-    <parent link="base_footprint"/>
-    <origin xyz="0 0 0.05" rpy="0 0 0"/>
-    <child link="base_1"/>
-  </joint-->
   <joint name="fixed" type="fixed">
     <parent link="base_footprint"/>
@@ -91,11 +70,11 @@
     </inertial>
   </link>
-  <joint name="joint1" type="continuous">
+  <joint name="joint1" type="revolute">
     <parent link="link1"/>
     <child link="link2"/>
     <origin xyz="0 ${width} ${height1 - axel_offset}" rpy="0 0 0"/>
     <axis xyz="0 1 0"/>
-    <dynamics damping="0.7"/>
-    <limit velocity="10000" effort="10000" lower="0" upper="1" />
+    <dynamics damping="0.1"/>
+    <limit velocity="10000" effort="10000" lower="${-PI/6}" upper="${PI/6}" />
   </joint>
   <!-- Middle Link -->
@@ -123,88 +102,4 @@
     </inertial>
   </link>
-  <joint name="joint2" type="fixed">
-    <parent link="link2"/>
-    <child link="link3"/>
-    <origin xyz="0 ${width} ${height2 - axel_offset*2}" rpy="0 0 0"/>
-    <axis xyz="0 1 0"/>
-    <dynamics damping="0.7"/>
-  </joint>
-  <!-- Top Link -->
-  <link name="link3">
-    <collision>
-      <origin xyz="0 0 ${height3/2 - axel_offset}" rpy="0 0 0"/>
-      <geometry>
-	<box size="${width} ${width} ${height3}"/>
-      </geometry>
-    </collision>
-    <visual>
-      <origin xyz="0 0 ${height3/2 - axel_offset}" rpy="0 0 0"/>
-      <geometry>
-	<box size="${width} ${width} ${height3}"/>
-      </geometry>
-      <material name="orange"/>
-    </visual>
-    <inertial>
-      <origin xyz="0 0 ${height3/2 - axel_offset}" rpy="0 0 0"/>
-      <mass value="${mass}"/>
-      <inertia
-	  ixx="${mass / 12.0 * (width*width + height3*height3)}" ixy="0.0" ixz="0.0"
-	  iyy="${mass / 12.0 * (height3*height3 + width*width)}" iyz="0.0"
-	  izz="${mass / 12.0 * (width*width + width*width)}"/>
-    </inertial>
-  </link>
-  <joint name="hokuyo_joint" type="fixed">
-    <axis xyz="0 1 0" />
-    <origin xyz="0 0 ${height3 - axel_offset/2}" rpy="0 0 0"/>
-    <parent link="link3"/>
-    <child link="hokuyo_link"/>
-  </joint>
-  <!-- Hokuyo Laser -->
-  <link name="hokuyo_link">
-    <collision>
-      <origin xyz="0 0 0" rpy="0 0 0"/>
-      <geometry>
-	<box size="0.1 0.1 0.1"/>
-      </geometry>
-    </collision>
-    <visual>
-      <origin xyz="0 0 0" rpy="0 0 0"/>
-      <geometry>
-        <mesh filename="package://rrbot_description/meshes/hokuyo.dae"/>
-      </geometry>
-    </visual>
-    <inertial>
-      <mass value="1e-5" />
-      <origin xyz="0 0 0" rpy="0 0 0"/>
-      <inertia ixx="1e-6" ixy="0" ixz="0" iyy="1e-6" iyz="0" izz="1e-6" />
-    </inertial>
-  </link>
-  <joint name="camera_joint" type="fixed">
-    <axis xyz="0 1 0" />
-    <origin xyz="${camera_link} 0 ${height3 - axel_offset*2}" rpy="0 0 0"/>
-    <parent link="link3"/>
-    <child link="camera_link"/>
-  </joint>
-  <!-- Camera -->
-  <link name="camera_link">
-    <collision>
-      <origin xyz="0 0 0" rpy="0 0 0"/>
-      <geometry>
-	<box size="${camera_link} ${camera_link} ${camera_link}"/>
-      </geometry>
-    </collision>
-    <visual>
-      <origin xyz="0 0 0" rpy="0 0 0"/>
-      <geometry>
-	<box size="${camera_link} ${camera_link} ${camera_link}"/>
-      </geometry>
-      <material name="red"/>
-    </visual>
-    <inertial>
-      <mass value="1e-5" />
-      <origin xyz="0 0 0" rpy="0 0 0"/>
-      <inertia ixx="1e-6" ixy="0" ixz="0" iyy="1e-6" iyz="0" izz="1e-6" />
-    </inertial>
-  </link>
   <transmission name="tran1">
     <type>transmission_interface/SimpleTransmission</type>
@@ -217,14 +112,4 @@
     </actuator>
   </transmission>
-  <!--transmission name="tran2">
-    <type>transmission_interface/SimpleTransmission</type>
-    <joint name="joint2">
-      <hardwareInterface>EffortJointInterface</hardwareInterface>
-    </joint>
-    <actuator name="motor2">
-      <hardwareInterface>EffortJointInterface</hardwareInterface>
-      <mechanicalReduction>1</mechanicalReduction>
-    </actuator>
-  </transmission-->
   <gazebo>
     <plugin name="object_controller" filename="libgazebo_ros_force_based_move.so">

Commit message: changed to gazebo7, lqr complited

File: environment/rrbot_description/urdf/rrbot.xacro (robot description, xacro)
@@ -5,7 +5,9 @@
   <xacro:property name="PI" value="3.1415926535897931"/>
   <xacro:property name="mass" value="0.2" /> <!-- arbitrary value for mass -->
-  <xacro:property name="width" value="0.1" /> <!-- Square dimensions (widthxwidth) of beams -->
-  <xacro:property name="height1" value="1.1" /> <!-- Link 1 -->
+  <xacro:property name="width" value="0.07" /> <!-- Square dimensions (widthxwidth) of beams -->
+  <xacro:property name="height1" value="0.8" /> <!-- Link 1 -->
   <xacro:property name="height2" value="0.6" /> <!-- Link 2 -->
+  <xacro:property name="height3" value="1" /> <!-- Link 3 -->
+  <xacro:property name="camera_link" value="0.05" /> <!-- Size of square 'camera' box -->
   <xacro:property name="axel_offset" value="0.05" /> <!-- Space btw top of beam and the each joint -->
   <!-- Import all Gazebo-customization elements, including Gazebo colors -->
@@ -19,5 +21,5 @@
       <origin xyz="0 0 0.01" rpy="0 0 0" />
       <geometry>
-        <box size="2.00 2.00 0.1" />
+        <box size="1.00 0.70 0.2" />
       </geometry>
     </visual>
@@ -31,5 +33,8 @@
       <origin xyz="0 0 0.02" rpy="0 0 0"/>
       <mass value="0.5"/>
-      <inertia ixx="1000" ixy="1000" ixz="1000" iyy="1000" iyz="1000" izz="1000" />
+      <inertia
+	  ixx="${mass / 12.0 * (width*width + height1*height1)}" ixy="0.0" ixz="0.0"
+	  iyy="${mass / 12.0 * (height1*height1 + width*width)}" iyz="0.0"
+	  izz="${mass / 12.0 * (width*width + width*width)}"/>
     </inertial>
   </link>
@@ -39,6 +44,25 @@
     <child link="base_footprint"/>
     <axis xyz="1 0 0"/>
-    <limit velocity="10000" effort="10000" lower="-10" upper="10" />
+    <limit velocity="1" effort="0.01" lower="-10" upper="10" />
   </joint>
+ <!-- link name="base_1">
+   <visual>
+      <origin xyz="1 0 1.51" rpy="0 0 0" />
+      <geometry>
+        <box size="0.1 2.1 3" />
+      </geometry>
+    </visual>
+   <collision>
+      <origin xyz="1 0 1.51" rpy="0 0 0" />
+      <geometry>
+        <box size="0.1 2.1 3" />
+      </geometry>
+    </collision>
+  </link >
+  <joint name="f_1" type="fixed">
+    <parent link="base_footprint"/>
+    <origin xyz="0 0 0.05" rpy="0 0 0"/>
+    <child link="base_1"/>
+  </joint-->
   <joint name="fixed" type="fixed">
     <parent link="base_footprint"/>
@@ -76,5 +100,5 @@
     <axis xyz="0 1 0"/>
     <dynamics damping="0.1"/>
-    <limit velocity="10000" effort="10000" lower="${-PI/6}" upper="${PI/6}" />
+    <limit velocity="10000" effort="10000" lower="${-PI}" upper="${PI}" />
   </joint>
   <!-- Middle Link -->
@@ -109,7 +133,10 @@
     <actuator name="motor1">
       <hardwareInterface>EffortJointInterface</hardwareInterface>
-      <mechanicalReduction>1</mechanicalReduction>
+      <mechanicalReduction>100</mechanicalReduction>
     </actuator>
   </transmission>
+  <plugin name="gazebo_ros_control" filename="libgazebo_ros_control.so">
+    <robotNamespace>/rrbot</robotNamespace>
+  </plugin>
   <gazebo>
     <plugin name="object_controller" filename="libgazebo_ros_force_based_move.so">
